File: _autosave-eeg.sch (KiCad schematic (older format))
At the start: 132 parts, among them J1 Conn_01x05_Male, J10 USB_B_Mini, J2 Conn_01x05_Male, J3 Conn_01x05_Male, J4 Conn_01x05_Male, J5 Conn_01x10, J6 Conn_01x10_Male, J7 Conn_01x10_Male, SW3 EVQ-Q2K03W, U1 STM32F446RE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

Commit message: RN4678's mode switch added
Parts:
- added R23, R24, R25: R_Small, symbol Device:R_Small
- added SW?: SW_DIP_x03, symbol Switch:SW_DIP_x03
Connections:
- net labels added: EAN, P2.0, P2.4
- wire segments 430 -> 433
- no-connect marks 60 -> 57
