File: eeg.sch (KiCad schematic (older format))
At the start: 132 parts, among them J1 Conn_01x05_Male, J10 USB_B_Mini, J2 Conn_01x05_Male, J3 Conn_01x05_Male, J4 Conn_01x05_Male, J5 Conn_01x10, J6 Conn_01x10_Male, J7 Conn_01x10_Male, SW3 EVQ-Q2K03W, U1 STM32F446RE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

Commit message: RN4678's SW_BTN added
Parts:
- added R23: 10R, symbol Device:R_Small
- added R24, R25: 4.7K, symbol Device:R_Small
- added SW2: SW_DIP_x03, Button_Switch_SMD:SW_DIP_SPSTx03_Slide_6.7x9.18mm_W6.73mm_P2.54mm_LowProfile_JPin, symbol Switch:SW_DIP_x03
Connections:
- net labels added: EAN, GND, INT3V3, P2.0, P2.4
- wire segments 430 -> 443
- no-connect marks 60 -> 57
